File: hardware/Ponder.kicad_sch (KiCad schematic)
At the start: 0 parts

Commit message: Updating template for project
Other:
- title: Top Level -> Ponder
Changed lines of the file:
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@@
   (paper "A3")
   (title_block
-    (title "Top Level")
-    (date "2024-02-29")
+    (title "Ponder")
+    (date "2024-09-03")
     (rev "0.1")
   )

Commit message: Adding baseline MCU and supportive blocks
Parts:
- added C1, C6: 10u, Capacitor_SMD:C_0805_2012Metric, symbol Device:C
- added C10, C11, C7, C8: 4.7u, Capacitor_SMD:C_0402_1005Metric, symbol Device:C
- added C12, C13, C14, C15, C16, C17, C18, C19, C2, C21, C3, C9: 100n, Capacitor_SMD:C_0402_1005Metric, symbol Device:C
- added C4, C5: 15p, Capacitor_SMD:C_0402_1005Metric, symbol Device:C
- added H1, H2, H3, H4: MountingHole, MountingHole:MountingHole_2.7mm_M2.5, symbol Mechanical:MountingHole
- added J3: SM03B-SRSS-TB, Connector_JST:JST_SH_SM03B-SRSS-TB_1x03-1MP_P1.00mm_Horizontal, symbol Connector_Generic_MountingPin:Conn_01x03_MountingPin
- added J5: USB_C_Receptacle_USB2.0, symbol Connector:USB_C_Receptacle_USB2.0
- added L1: 3.3u, Ponder:L_pol_2016, symbol Device:L
- added R1, R2, R3: 1k, Resistor_SMD:R_0402_1005Metric, symbol Device:R
- added R10, R11: 27, Resistor_SMD:R_0402_1005Metric, symbol Device:R
- added R4: OMIT, Resistor_SMD:R_0402_1005Metric, symbol Device:R
- added R5, R6: 5k1, Resistor_SMD:R_0402_1005Metric, symbol Device:R
- added R8: 33, Resistor_SMD:R_0402_1005Metric, symbol Device:R
- added SW1, SW3: SW_Push, Button_Switch_SMD:SW_Push_1P1T_NO_Vertical_Wuerth_434133025816, symbol Switch:SW_Push
- added U1: W25Q128JVS, Package_SO:SOIC-8_5.23x5.23mm_P1.27mm, symbol Memory_Flash:W25Q128JVS
- added U3: NCP1117-3.3_SOT223, Package_TO_SOT_SMD:SOT-223-3_TabPin2, symbol Regulator_Linear:NCP1117-3.3_SOT223
- added U4: RP2350_80QFN, Ponder:RP2350-QFN-80-1EP_10x10_P0.4mm_EP3.4x3.4mm_ThermalVias, symbol Ponder:RP2350_80QFN
- added Y1: ABM8-272-T3, Crystal:Crystal_SMD_3225-4Pin_3.2x2.5mm, symbol Device:Crystal_GND24
Connections:
- new net: R1.1, SW1.1
- new net: R11.2, U4.66 (USB_DM)
- new net: C5.1, R2.2, Y1.3
- new net: R10.2, U4.67 (USB_DP)
- new net: J5.A5 (CC1), R5.2
- new net: J5.B5 (CC2), R6.2
- new net +1V1: C11.1, C12.1, C8.1, C9.1, L1.1, U4.10 (DVDD), U4.32 (DVDD), U4.51 (DVDD), U4.65 (VREG_FB)
- new net +3V3: C13.1, C14.1, C15.1, C16.1, C17.1, C18.1, C19.1, C2.1, C21.1, C3.1, C6.1, C7.1, R4.1, R8.1, U1.8 (VCC), U3.2 (VO), U4.15 (IOVDD), U4.24 (IOVDD), U4.29 (IOVDD), U4.41 (IOVDD), U4.5 (IOVDD), U4.50 (IOVDD), U4.59 (ADC_AVDD), U4.60 (IOVDD), U4.64 (VREG_VIN), U4.68 (USB_OTP_VDD), U4.69 (QSPI_IOVDD), U4.76 (IOVDD)
- new net GND: C1.2, C10.2, C11.2, C12.2, C13.2, C14.2, C15.2, C16.2, C17.2, C18.2, C19.2, C2.2, C21.2, C3.2, C4.2, C5.2, C6.2, C7.2, C8.2, C9.2, J3.2 (Pin_2), J3.MP (MountPin), J5.A1 (GND), J5.A12 (GND), J5.B1 (GND), J5.B12 (GND), J5.S1 (SHIELD), R1.2, R5.1, R6.1, SW3.1, U1.4 (GND), U3.1 (GND), U4.62 (VREG_PGND), U4.81 (GND), Y1.2, Y1.4
- new net GPIO0: U4.77 (GPIO0)
- new net GPIO1: U4.78 (GPIO1)
- new net GPIO10: U4.8 (GPIO10)
- new net GPIO11: U4.9 (GPIO11)
- new net GPIO12: U4.11 (GPIO12)
- new net GPIO13: U4.12 (GPIO13)
- new net GPIO14: U4.13 (GPIO14)
- new net GPIO15: U4.14 (GPIO15)
- new net GPIO16: U4.16 (GPIO16)
- new net GPIO17: U4.17 (GPIO17)
- new net GPIO18: U4.18 (GPIO18)
- new net GPIO19: U4.19 (GPIO19)
- new net GPIO2: U4.79 (GPIO2)
- new net GPIO20: U4.20 (GPIO20)
- new net GPIO21: U4.21 (GPIO21)
- new net GPIO22: U4.22 (GPIO22)
- new net GPIO23: U4.23 (GPIO23)
- new net GPIO24: U4.25 (GPIO24)
- new net GPIO25: U4.26 (GPIO25)
- new net GPIO26: U4.27 (GPIO26)
- new net GPIO27: U4.28 (GPIO27)
- new net GPIO28: U4.36 (GPIO28)
- new net GPIO29: U4.37 (GPIO29)
- new net GPIO3: U4.80 (GPIO3)
- new net GPIO30: U4.38 (GPIO30)
- new net GPIO31: U4.39 (GPIO31)
- new net GPIO32: U4.40 (GPIO32)
- new net GPIO33: U4.42 (GPIO33)
- new net GPIO34: U4.43 (GPIO34)
- new net GPIO35: U4.44 (GPIO35)
- new net GPIO36: U4.45 (GPIO36)
- new net GPIO37: U4.46 (GPIO37)
- new net GPIO38: U4.47 (GPIO38)
- new net GPIO39: U4.48 (GPIO39)
- new net GPIO4: U4.1 (GPIO4)
- new net GPIO40_ADC0: U4.49 (GPIO40_ADC0)
- new net GPIO41_ADC1: U4.52 (GPIO41_ADC1)
- new net GPIO42_ADC2: U4.53 (GPIO42_ADC2)
- new net GPIO43_ADC3: U4.54 (GPIO43_ADC3)
- new net GPIO44_ADC4: U4.55 (GPIO44_ADC4)
- new net GPIO45_ADC5: U4.56 (GPIO45_ADC5)
- new net GPIO46_ADC6: U4.57 (GPIO46_ADC6)
- new net GPIO47_ADC7: U4.58 (GPIO47_ADC7)
- new net GPIO5: U4.2 (GPIO5)
- new net GPIO6: U4.3 (GPIO6)
- new net GPIO7: U4.4 (GPIO7)
- new net GPIO8: U4.6 (GPIO8)
- new net GPIO9: U4.7 (GPIO9)
- new net QSPI_SCLK: U1.6 (CLK), U4.71 (QSPI_SCLK)
- new net QSPI_SD0: U1.5 (DI(IO0)), U4.72 (QSPI_SD0)
- new net QSPI_SD1: U1.2 (DO(IO1)), U4.74 (QSPI_SD1)
- new net QSPI_SD2: U1.3 (IO2), U4.73 (QSPI_SD2)
- new net QSPI_SD3: U1.7 (IO3), U4.70 (QSPI_SD3)
- new net QSPI_SS: R3.1, R4.2, U1.1 (~{CS}), U4.75 (QSPI_SS)
- new net RUN: SW1.2, U4.35 (RUN)
- new net SWCLK: J3.1 (Pin_1), U4.33 (SWCLK)
- new net SWD: J3.3 (Pin_3), U4.34 (SWD)
- new net USB_D+: J5.A6 (D+), J5.B6 (D+), R10.1
- new net USB_D-: J5.A7 (D-), J5.B7 (D-), R11.1
- new net VBUS: C1.1, J5.A4 (VBUS), J5.A9 (VBUS), J5.B4 (VBUS), J5.B9 (VBUS), U3.3 (VI)
- new net VREG_AVDD: C10.1, R8.2, U4.61 (VREG_AVDD)
- new net VREG_LX: L1.2, U4.63 (VREG_LX)
- new net XIN: C4.1, U4.30 (XIN), Y1.1
- new net XOUT: R2.1, U4.31 (XOUT)
- new net ~{USB_BOOT}: R3.2, SW3.2
- no-connect marks 0 -> 2
Other:
- note added: "Board Furniture"
- note added: "Boot / Flash"
- note added: "Configuration"
- note added: "External Power"
- note added: "Interfaces"
- note added: "JST Debug Connector"
- note added: "MCU"
- note added: "Note: Place Rs close to P67,66"
- note added: "Note: Place close to DVDD pins"
- note added: "Note: Place close to IOVDD pins"
- note added: "Note: Shenannigans on internal DCDC... DS "6.3.8.3. Regulator Sensitivities""
- note added: "Power Rails"
- note added: "Programming"
- note added: "Rail decoupling"
- note added: "Reset"

Commit message: Adding programming headers, some testpoints, and minimal MCU fanout with power
Parts:
- added J3: Conn_ARM_JTAG_SWD_10, Connector_PinHeader_1.27mm:PinHeader_2x05_P1.27mm_Vertical_SMD, symbol Connector:Conn_ARM_JTAG_SWD_10
- added TP1, TP10, TP11, TP2, TP3, TP4, TP5, TP6, TP7, TP8, TP9: TestPoint, TestPoint:TestPoint_Pad_D1.0mm, symbol Connector:TestPoint
- J1: renamed from J5; footprint (none) -> Connector_USB:USB_C_Receptacle_GCT_USB4105-xx-A_16P_TopMnt_Horizontal
- renumbered C9 to C1, C18 to C10, C19 to C11, C21 to C12, C1 to C13, C6 to C14, C10 to C15, C7 to C16, C8 to C17, C2 to C18, C4 to C19, C11 to C2, C5 to C20, C12 to C3, C3 to C4, C13 to C5, C14 to C6, C15 to C7, C16 to C8, C17 to C9, J3 to J2, R5 to R1, R6 to R2, R8 to R3, R1 to R4, R10 to R5, R11 to R6, R4 to R7, R3 to R8, R2 to R9, SW3 to SW2, U3 to U1, U1 to U2, U4 to U3, Y1 to X1
Connections:
- net +1V1: now also TP6.1
- net +3V3: now also J3.1 (VTref), TP10.1, TP2.1
- net GND: now also J3.3 (GND), J3.5 (GND), TP3.1, TP4.1, TP5.1, TP9.1
- net RUN: now also J3.10 (~{RESET}), TP11.1
- net SWCLK: now also J3.4 (SWDCLK/TCK), TP7.1
- net SWD: now also J3.2 (SWDIO/TMS), TP8.1
- net VBUS: now also TP1.1
- no-connect marks 2 -> 4
Other:
- note added: "Note: ARM Debug"
- note added: "Note: JST Debug"
- note added: "Note: Test Points"
- note removed: "JST Debug Connector"
- moved on the sheet: C14, J2
