File: hardware/Ponder.kicad_pcb (KiCad board)
At the start: 2 copper layers, 40 x 50 mm, 136 parts, among them J1 USB_C_Receptacle_USB2.0, J10 2.54 SKT, J11 2.54 HDR, J12 1.27 HDR, J13 1.27 HDR, J14 1.27 HDR, J15 1.27 HDR, J2 2.54 HDR, J3 2.54 HDR, J4 2.54 HDR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

Commit message: Unifying vias to single drill. Adding some plane connections
Routing:
- net +3V3: track 73.5 -> 80.4 mm, vias 13 -> 17
- net /RUN: track 46.6 -> 49.1 mm
