File: hardware/Ponder-Pico2.kicad_sch (KiCad schematic)
At the start: 136 parts, among them J1 USB_C_Receptacle_USB2.0, J10 2.54 SKT, J11 2.54 HDR, J12 1.27 HDR, J13 1.27 HDR, J14 1.27 HDR, J15 1.27 HDR, J2 2.54 HDR, J3 2.54 HDR, J4 2.54 HDR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

Commit message: Adding start of Pico 2 variant for Ponder
Parts:
- removed C1, C10, C11, C12, C18, C3, C4, C5, C6, C7, C8, C9: 100n, Capacitor_SMD:C_0402_1005Metric, symbol Device:C
- removed C14: 10u, Capacitor_SMD:C_0805_2012Metric, symbol Device:C
- removed C15, C2: 4.7u, Capacitor_SMD:C_0402_1005Metric, symbol Device:C
- removed C16, C17: 4.7u, Ponder:C_0402_1005Metric_small_pads, symbol Device:C
- removed C19, C20: 15p, Capacitor_SMD:C_0402_1005Metric, symbol Device:C
- removed J11: 2.54 HDR, Connector_PinHeader_2.54mm:PinHeader_1x04_P2.54mm_Vertical_SMD_Pin1Left, symbol Connector_Generic:Conn_01x04
- removed L1: 3.3u, Ponder:L_pol_2016, symbol Device:L
- removed R3: 33, Resistor_SMD:R_0402_1005Metric, symbol Device:R
- removed R5, R6: 27, Resistor_SMD:R_0402_1005Metric, symbol Device:R
- removed R9: 1k, Resistor_SMD:R_0402_1005Metric, symbol Device:R
- removed TP10, TP11, TP12, TP6, TP7, TP8, TP9: TestPoint, TestPoint:TestPoint_Pad_D1.0mm, symbol Connector:TestPoint
- removed U1: NCP1117-3.3_SOT223, Package_TO_SOT_SMD:SOT-223-3_TabPin2, symbol Regulator_Linear:NCP1117-3.3_SOT223
- removed U2: W25Q64JVXGIQ_TR, Ponder:SON80P400X400X50-9N, symbol Memory_Flash:W25Q128JVS
- removed U3: RP2350_80QFN, Ponder:RP2350-QFN-80-1EP_10x10_P0.4mm_EP3.4x3.4mm_ThermalVias, symbol Ponder:RP2350_80QFN
- removed X1: ABM8-272-T3, Crystal:Crystal_SMD_3225-4Pin_3.2x2.5mm, symbol Device:Crystal_GND24
- added H5, H6: MountingHole, MountingHole:MountingHole_2.7mm_M2.5, symbol Mechanical:MountingHole
- added U1: ~, Ponder:RaspberryPi-Pico-SMD-TP, symbol Ponder:RaspberryPi-Pico2
Connections:
- net +3V3: now also U1.36 (3V3(OUT))
- net GND: now also U1.13 (GND), U1.18 (GND), U1.23 (GND), U1.28 (GND), U1.3 (GND), U1.33 (GND), U1.38 (GND), U1.42 (GND), U1.44 (GND), U1.8 (GND)
- net RP_PWR_LED: now also U1.48 (GPIO25/LED)
- net RP_UART0_LED: now also U1.4 (GP2)
- net RP_UART0_RX: now also U1.2 (GP1)
- net RP_UART0_TX: now also U1.1 (GP0)
- net RP_UART1_LED: now also U1.9 (GP6)
- net RP_UART1_RX: now also U1.7 (GP5)
- net RP_UART1_TX: now also U1.6 (GP4)
- net RP_UART2_LED: now also U1.10 (GP7)
- net RP_UART2_RX: now also U1.12 (GP9)
- net RP_UART2_TX: now also U1.11 (GP8)
- net RP_UART3_LED: now also U1.15 (GP11)
- net RP_UART3_RX: now also U1.17 (GP13)
- net RP_UART3_TX: now also U1.16 (GP12)
- net RP_UART4_LED: now also U1.29 (GP22)
- net RP_UART4_RX: now also U1.26 (GP20)
- net RP_UART4_TX: now also U1.27 (GP21)
- net RP_UART5_LED: now also U1.34 (GP28)
- net RP_UART5_RX: now also U1.31 (GP26)
- net RP_UART5_TX: now also U1.32 (GP27)
- net RUN: now also U1.30 (RUN)
- net SWCLK: now also U1.41 (SWCLK)
- net SWD: now also U1.43 (SWDIO)
- net USB_D+: now also U1.46 (USB_DP)
- net USB_D-: now also U1.45 (USB_DM)
- net USR_SW: now also U1.5 (GP3)
- net VBUS: now also U1.40 (VBUS)
- net QSPI_SS renamed BOOTSEL
- net BOOTSEL: now also U1.49 (BOOTSEL)
- net RP_SPI1-CSn_I2C0-SCL renamed RP_SPI0-CSn_I2C0-SCL
- net RP_SPI0-CSn_I2C0-SCL: now also U1.22 (GP17)
- net RP_SPI1-MISO_I2C0-SDA renamed RP_SPI0-MISO_I2C0-SDA
- net RP_SPI0-MISO_I2C0-SDA: now also U1.21 (GP16)
- net RP_SPI1-MOSI_I2C1-SCL renamed RP_SPI0-MOSI_I2C1-SCL
- net RP_SPI0-MOSI_I2C1-SCL: now also U1.25 (GP19)
- net RP_SPI1-SCK_I2C1-SDA renamed RP_SPI0-SCK_I2C1-SDA
- net RP_SPI0-SCK_I2C1-SDA: now also U1.24 (GP18)
- no-connect marks 15 -> 10
Other:
- note removed: "Note: Place Rs close to P67,66"
- note removed: "Note: Place close to DVDD pins"
- note removed: "Note: Place close to IOVDD pins"
- note removed: "Note: Shenannigans on internal DCDC... DS "6.3.8.3. Regulator Sensitivities""
- title: Ponder -> Ponder-Pico2
